File: RaspberryPi_Connections.brd (EAGLE design)
At the start: 124.4 x 101.3 mm, 4 parts

Commit message: Final update before printing first prototype
Parts:
- moved PCB1 75.2 mm to (-10.2, -63.5)
- moved JP1 68.4 mm to (14.0, 8.89)
- moved JP2 68.4 mm to (11.4, 35.6)
- moved U$1 68.4 mm to (29.2, 19.1)
Routing:
- net TOOL_CHANGER_ANALOG_I: track 21.2 -> 23.3 mm
- net SCLK_A: track 28.2 -> 29.3 mm
- net MISO_A: track 36.2 -> 37.2 mm
- added copper zone on layer 1, net GND_RPI
Other:
- board size 124.4 x 101.3 mm -> 36.8 x 45.4 mm

Commit message: update
Parts:
- removed PCB1: RPI2, e14_Rpi2_RevA:RPI2
Changed lines of the file:
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@@
 </autorouter>
 <elements>
-<element name="PCB1" library="e14_Rpi2_RevA" package="RPI2" value="RPI2" x="-10.16" y="-63.5" smashed="yes"/>
 <element name="JP2" library="pinhead" library_urn="urn:adsk.eagle:library:325" package="1X05" package3d_urn="urn:adsk.eagle:package:22469/2" value="" x="11.43" y="35.56" smashed="yes">
 <attribute name="NAME" x="5.0038" y="37.3888" size="1.27" layer="25" ratio="10"/>
