File: ArduinoUNO_Connexions.brd (EAGLE design)
At the start: 167.6 x 130.8 mm, 73 parts

Commit message: update with new guidlines
Parts:
- added D3, D4, D5: 1N4004, diode:DO41-10
- added R20, R21, R22, R23, R24: 1k, rcl:0207/7
- added SV5: (no value), con-lstb:MA05-1
- added X1: (no value), con-ptr500:AK500/2
- R16: value 100k -> 0
- moved C6 129.5 mm to (139.7, 105.4)
- moved JP21 129.5 mm to (148.6, 83.8)
- moved JP22 129.5 mm to (148.6, 96.5)
- moved JP23 129.5 mm to (151.1, 76.2)
- moved JP24 129.5 mm to (148.6, 113.0)
- moved C7 128.3 mm to (30.5, 100.3), turned to 0 degrees
- moved C12 125.8 mm to (157.5, 100.3), turned to 0 degrees
- moved JP1 124.5 mm to (21.6, 83.8)
- moved JP2 124.5 mm to (21.6, 96.5)
- moved JP3 124.5 mm to (21.6, 113.0)
- moved JP4 124.5 mm to (24.1, 76.2)
- moved C1 124.5 mm to (12.7, 105.4)
- moved JP19 78.7 mm to (125.7, 76.2)
- moved C5 78.7 mm to (114.3, 105.4)
- moved JP17 78.7 mm to (123.2, 83.8)
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Connections:
- new net A3: R22.1, SV3.4, SV5.3
- new net A4: R23.1, SV3.5, SV5.4
- new net A5: R24.1, SV3.6, SV5.5
- new net D12: R20.2, SV4.5, SV5.1
- new net D13: R21.2, SV4.6, SV5.2
- new net N$56: D4.A, D5.A, X1.2
- net DIR$0: now also R1.2, SV1.1; no longer R2.2, SV1.2
- net DIR$1: now also R3.2, SV1.3; no longer R4.2, SV1.4
- net DIR$2: now also R5.2, SV1.5; no longer R6.2, SV1.6
- net DIR$3: now also R7.2, SV1.7; no longer R8.2, SV1.8
- net DIR$4: now also R9.2, SV4.1; no longer R10.2, SV4.2
- net DIR$5: now also R11.2, SV4.3; no longer R12.2, SV4.4
- net GND: now also R20.1, R21.1, R22.2, R23.2, R24.2
- net GNDMOT: now also X1.1
- net N$1: now also D3.A; no longer LED3.A
- net N$2: now also D1.A; no longer D1.C
- net STEP$0: now also R2.2, SV1.2; no longer R1.2, SV1.1
- net STEP$1: now also R4.2, SV1.4; no longer R3.2, SV1.3
- net STEP$2: now also R6.2, SV1.6; no longer R5.2, SV1.5
- net STEP$3: now also R8.2, SV1.8; no longer R7.2, SV1.7
- net STEP$4: now also R10.2, SV4.2; no longer R9.2, SV4.1
- net STEP$5: now also R12.2, SV4.4; no longer R11.2, SV4.3
- net VCC: now also D1.C; no longer D1.A
- net VMOT: now also D3.C, D4.C, D5.C, LED3.A
Routing:
- net N$1: track 147.7 -> 0.00 mm
- net A3: track 0.00 -> 117.3 mm
- net VMOT: track 0.00 -> 113.0 mm
- net A4: track 0.00 -> 109.7 mm
- net A5: track 0.00 -> 99.5 mm
- net RESOLUTION$2: track 282.6 -> 356.5 mm, vias 0 -> 6
- net D12: track 0.00 -> 68.4 mm
- net D13: track 0.00 -> 64.8 mm
- net RESOLUTION$1: track 311.2 -> 341.7 mm, vias 5 -> 6
- net GND: track 29.2 -> 0.00 mm
- net STEP$4: track 52.3 -> 75.2 mm
- net DIR$4: track 52.5 -> 75.1 mm
- net DIR$0: track 67.4 -> 45.7 mm
- net STEP$3: track 34.7 -> 55.7 mm
- net STEP$0: track 67.4 -> 46.7 mm
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- added copper zone on layer 1, net N$1
- added copper zone on layer 1, net N$56
- removed copper zone on layer 1, net DIR$5

Commit message: Final update before printing first prototype
Parts:
- added S1: (no value), switch:255SB
- moved PCB2 56.0 mm to (106.7, -76.2), flipped to the bottom
Connections:
- new net N$43: S1.2, SV2.1
- net VCC: now also S1.1
Routing:
- net N$43: track 0.00 -> 89.4 mm, vias 0 -> 1
- net VCC: track 210.7 -> 239.0 mm
- net N$2: track 37.7 -> 44.1 mm
- net N$3: track 102.1 -> 105.2 mm

Commit message: Update
Parts:
- added D6: (no value), diode:F126Z12
- added X2: (no value), con-ptr500:AK500/2
- moved D1 16.1 mm to (3.81, 77.5)
- moved X3 1.27 mm to (7.62, 47.0), turned to 270 degrees
- flipped X1 to the top, turned to 180 degrees
Connections:
- new net ALIM_ARDUINO: D6.C, S1.1
- new net N$44: D6.A, X2.2
- net GND: now also X2.1
- net VCC: no longer S1.1
Routing:
- net VCC: track 239.0 -> 199.0 mm
- net N$2: track 44.1 -> 53.2 mm
- net N$44: track 0.00 -> 8.90 mm
- net ALIM_ARDUINO: track 0.00 -> 5.61 mm
Other:
- board text added: "5V"
- board text added: "Alim Arduino (Vin)"
- board text added: "Arduino UNO Shield"
- board text added: "Board - USB"
- board text added: "VMOT"
- board text removed: "5V Board"

Commit message: update
Parts:
- removed PCB2: ARDUINO_UNO, E14_Arduino_revC:ARDUINO_UNO
- removed U$1, U$2, U$3, U$4, U$5, U$6: BOARD_A4988, Clean-Kong:BOARD_A4988
Connections:
- removed net VDD: U$1.+5V, U$2.+5V, U$3.+5V, U$4.+5V, U$5.+5V, U$6.+5V
- net GND: no longer U$1.GND, U$2.GND, U$3.GND, U$4.GND, U$5.GND, U$6.GND
- net GNDMOT: no longer U$1.GNDMOT, U$2.GNDMOT, U$3.GNDMOT, U$4.GNDMOT, U$5.GNDMOT, U$6.GNDMOT
- net VMOT: no longer U$1.VMOT, U$2.VMOT, U$3.VMOT, U$4.VMOT, U$5.VMOT, U$6.VMOT
Other:
- board text added: "Increase mounting holes mask size for the screw head"
Changed lines of the file:
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@@
 <text x="121.92" y="123.19" size="1.778" layer="21">VMOT</text>
 <text x="87.63" y="38.1" size="1.778" layer="21">Arduino UNO Shield</text>
+<text x="-2.54" y="133.35" size="1.778" layer="51">Increase mounting holes mask size for the screw head</text>
+<text x="158.75" y="133.35" size="1.778" layer="51">Increase mounting holes mask size for the screw head</text>
+<text x="-7.62" y="-5.08" size="1.778" layer="51">Increase mounting holes mask size for the screw head</text>
+<text x="160.02" y="-3.81" size="1.778" layer="51">Increase mounting holes mask size for the screw head</text>
 </plain>
 <attributes>
@@
 </autorouter>
 <elements>
-<element name="PCB2" library="E14_Arduino_revC" package="ARDUINO_UNO" value="ARDUINO_UNO" x="106.68" y="-76.2" smashed="yes" rot="MR0"/>
 <element name="R1" library="rcl" library_urn="urn:adsk.eagle:library:334" package="0207/7" package3d_urn="urn:adsk.eagle:package:23493/1" value="1k" x="54.61" y="52.07" smashed="yes" rot="R90">
 <attribute name="NAME" x="54.483" y="44.45" size="1.27" layer="25" ratio="10" rot="R90"/>
@@
 <attribute name="AMPS" value="15" x="21.59" y="125.73" size="1.778" layer="27" display="off"/>
 <attribute name="NAME" x="19.558" y="127.381" size="1.27" layer="25" ratio="10"/>
-</element>
-<element name="U$1" library="Clean-Kong" package="BOARD_A4988" value="BOARD_A4988" x="-35.56" y="82.55" smashed="yes">
-<attribute name="NAME" x="-30.48" y="95.25" size="1.27" layer="25"/>
-</element>
-<element name="U$2" library="Clean-Kong" package="BOARD_A4988" value="BOARD_A4988" x="-52.07" y="82.55" smashed="yes">
-<attribute name="NAME" x="-46.99" y="95.25" size="1.27" layer="25"/>
-</element>
-<element name="U$3" library="Clean-Kong" package="BOARD_A4988" value="BOARD_A4988" x="-68.58" y="82.55" smashed="yes">
-<attribute name="NAME" x="-63.5" y="95.25" size="1.27" layer="25"/>
-</element>
-<element name="U$4" library="Clean-Kong" package="BOARD_A4988" value="BOARD_A4988" x="-85.09" y="82.55" smashed="yes">
-<attribute name="NAME" x="-80.01" y="95.25" size="1.27" layer="25"/>
-</element>
-<element name="U$5" library="Clean-Kong" package="BOARD_A4988" value="BOARD_A4988" x="-101.6" y="82.55" smashed="yes">
-<attribute name="NAME" x="-96.52" y="95.25" size="1.27" layer="25"/>
-</element>
-<element name="U$6" library="Clean-Kong" package="BOARD_A4988" value="BOARD_A4988" x="-118.11" y="82.55" smashed="yes">
-<attribute name="NAME" x="-113.03" y="95.25" size="1.27" layer="25"/>
 </element>
 <element name="LED1" library="led" library_urn="urn:adsk.eagle:library:259" package="LED5MM" package3d_urn="urn:adsk.eagle:package:15799/2" value="" x="10.16" y="33.02" smashed="yes">
@@
 <contactref element="C12" pad="2"/>
 <contactref element="X3" pad="1"/>
-<contactref element="U$1" pad="GND"/>
-<contactref element="U$2" pad="GND"/>
-<contactref element="U$3" pad="GND"/>
-<contactref element="U$4" pad="GND"/>
-<contactref element="U$5" pad="GND"/>
-<contactref element="U$6" pad="GND"/>
 <contactref element="R17" pad="1"/>
 <contactref element="R18" pad="2"/>
@@
 </polygon>
 <contactref element="X2" pad="1"/>
-<wire x1="-50.8" y1="101.6" x2="-34.29" y2="101.6" width="0" layer="19" extent="1-1"/>
-<wire x1="-67.31" y1="101.6" x2="-50.8" y2="101.6" width="0" layer="19" extent="1-1"/>
-<wire x1="-83.82" y1="101.6" x2="-67.31" y2="101.6" width="0" layer="19" extent="1-1"/>
-<wire x1="-100.33" y1="101.6" x2="-83.82" y2="101.6" width="0" layer="19" extent="1-1"/>
-<wire x1="-116.84" y1="101.6" x2="-100.33" y2="101.6" width="0" layer="19" extent="1-1"/>
-<wire x1="6.35" y1="90.17" x2="-34.29" y2="101.6" width="0" layer="19" extent="1-1"/>
 </signal>
 <signal name="VCC">
@@
 <contactref element="C6" pad="+"/>
 <contactref element="D2" pad="C"/>
-<contactref element="U$1" pad="VMOT"/>
-<contactref element="U$2" pad="VMOT"/>
-<contactref element="U$3" pad="VMOT"/>
-<contactref element="U$4" pad="VMOT"/>
-<contactref element="U$5" pad="VMOT"/>
-<contactref element="U$6" pad="VMOT"/>
 <contactref element="D4" pad="C"/>
 <contactref element="D3" pad="C"/>
@@
 <wire x1="1.27" y1="20.32" x2="8.89" y2="12.7" width="1.016" layer="1"/>
 <wire x1="1.27" y1="97.79" x2="1.27" y2="20.32" width="1.016" layer="1"/>
-<wire x1="-50.8" y1="83.82" x2="-34.29" y2="83.82" width="0" layer="19" extent="1-1"/>
-<wire x1="-67.31" y1="83.82" x2="-50.8" y2="83.82" width="0" layer="19" extent="1-1"/>
-<wire x1="-83.82" y1="83.82" x2="-67.31" y2="83.82" width="0" layer="19" extent="1-1"/>
-<wire x1="-100.33" y1="83.82" x2="-83.82" y2="83.82" width="0" layer="19" extent="1-1"/>
-<wire x1="-116.84" y1="83.82" x2="-100.33" y2="83.82" width="0" layer="19" extent="1-1"/>
-<wire x1="1.27" y1="97.79" x2="-34.29" y2="83.82" width="0" layer="19" extent="1-1"/>
 </signal>
 <signal name="GNDMOT">
@@
 <contactref element="C6" pad="-"/>
 <contactref element="X4" pad="1"/>
-<contactref element="U$1" pad="GNDMOT"/>
-<contactref element="U$2" pad="GNDMOT"/>
-<contactref element="U$3" pad="GNDMOT"/>
-<contactref element="U$4" pad="GNDMOT"/>
-<contactref element="U$5" pad="GNDMOT"/>
-<contactref element="U$6" pad="GNDMOT"/>
 <wire x1="15.24" y1="96.52" x2="15.24" y2="105.41" width="1.524" layer="1"/>
 <wire x1="40.64" y1="96.52" x2="40.64" y2="105.41" width="1.524" layer="1"/>
@@
 <vertex x="167.64" y="130.81"/>
 </polygon>
-<wire x1="-50.8" y1="86.36" x2="-34.29" y2="86.36" width="0" layer="19" extent="1-1"/>
-<wire x1="-67.31" y1="86.36" x2="-50.8" y2="86.36" width="0" layer="19" extent="1-1"/>
-<wire x1="-83.82" y1="86.36" x2="-67.31" y2="86.36" width="0" layer="19" extent="1-1"/>
-<wire x1="-100.33" y1="86.36" x2="-83.82" y2="86.36" width="0" layer="19" extent="1-1"/>
-<wire x1="-116.84" y1="86.36" x2="-100.33" y2="86.36" width="0" layer="19" extent="1-1"/>
-<wire x1="6.35" y1="97.79" x2="-34.29" y2="86.36" width="0" layer="19" extent="1-1"/>
 </signal>
 <signal name="N$5">
@@
 <contactref element="X4" pad="2"/>
 </signal>
-<signal name="VDD">
-<contactref element="U$1" pad="+5V"/>
-<contactref element="U$2" pad="+5V"/>
-<contactref element="U$3" pad="+5V"/>
-<contactref element="U$4" pad="+5V"/>
-<contactref element="U$5" pad="+5V"/>
-<contactref element="U$6" pad="+5V"/>
-<wire x1="-50.8" y1="99.06" x2="-34.29" y2="99.06" width="0" layer="19" extent="1-1"/>
-<wire x1="-67.31" y1="99.06" x2="-50.8" y2="99.06" width="0" layer="19" extent="1-1"/>
-<wire x1="-83.82" y1="99.06" x2="-67.31" y2="99.06" width="0" layer="19" extent="1-1"/>
-<wire x1="-100.33" y1="99.06" x2="-83.82" y2="99.06" width="0" layer="19" extent="1-1"/>
-<wire x1="-116.84" y1="99.06" x2="-100.33" y2="99.06" width="0" layer="19" extent="1-1"/>
-</signal>
 <signal name="N$3">

Commit message: update
Other:
- board text removed: "Increase mounting holes mask size for the screw head"

Commit message: update
Parts:
- removed R20, R21: 1k, rcl:0207/7
- added S2: (no value), switch-omron:B3F-10XX
- C1, C2, C3, C4, C5, C6: value (none) -> 100uF
- C10, C11, C12, C7, C8, C9: value (none) -> 0,1uF
- D2, D3, D4, D5: value 1N4004 -> 1N5400; device diode:DO41-10 -> diode:DO201-15
- R17, R18: value 250 -> 125
- R19: value 2,7K -> 1,4K
- SV5: device con-lstb:MA05-1 -> con-lstb:MA03-1
- moved D3 80.1 mm to (101.6, 119.4)
- moved D2 80.0 mm to (101.6, 125.7)
- moved D5 73.7 mm to (26.7, 119.4)
- moved D4 73.7 mm to (26.7, 125.7)
- moved X4 10.2 mm to (44.5, 124.5)
- moved R7 6.60 mm to (76.5, 52.1)
- moved R8 6.60 mm to (79.0, 52.1)
- moved R9 5.08 mm to (81.5, 52.1)
- moved R4 5.08 mm to (67.3, 52.1)
- moved R22 5.08 mm to (144.8, 24.1)
- moved R24 5.08 mm to (144.8, 29.2)
- moved R1 5.08 mm to (59.7, 52.1)
- moved R10 5.08 mm to (84.1, 52.1)
- moved R11 5.08 mm to (86.6, 52.1)
- moved R12 5.08 mm to (89.2, 52.1)
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Connections:
- net N$43 renamed VIN_ARDUINO
- removed net D12: R20.2, SV4.5, SV5.1
- removed net D13: R21.2, SV4.6, SV5.2
- removed net N$3: LED1.A, SV2.5
- new net 3V3_ARDUINO: SV2.5
- new net 5V_ARDUINO: LED1.A, SV2.4
- new net IOREF_ARDUINO: SV2.7
- new net RESET_ARDUINO: S2.3, S2.4, SV2.6
- new net RX_ARDUINO: SV1.1
- new net TX_ARDUINO: SV1.2
- net A4: now also SV5.2; no longer SV5.4
- net A5: now also SV5.1; no longer SV5.5
- net DIR$0: now also SV1.3; no longer SV1.1
- net DIR$1: now also SV1.5; no longer SV1.3
- net DIR$2: now also SV1.7; no longer SV1.5
- net DIR$3: now also SV4.1; no longer SV1.7
- net DIR$4: now also SV4.3; no longer SV4.1
- net DIR$5: now also SV4.5; no longer SV4.3
- net GND: now also S2.1, S2.2; no longer R20.1, R21.1
- net N$1: now also D4.A, D5.A; no longer D2.A, D3.A
- net N$56: now also D2.A, D3.A; no longer D4.A, D5.A
- net STEP$0: now also SV1.4; no longer SV1.2
- net STEP$1: now also SV1.6; no longer SV1.4
- net STEP$2: now also SV1.8; no longer SV1.6
- net STEP$3: now also SV4.2; no longer SV1.8
- net STEP$4: now also SV4.4; no longer SV4.2
- net STEP$5: now also SV4.6; no longer SV4.4
Routing:
- net GND: track 0.00 -> 113.9 mm, vias 0 -> 31
- net 5V_ARDUINO: track 0.00 -> 105.4 mm, vias 0 -> 2
- net N$3: track 105.2 -> 0.00 mm, vias 1 -> 0
- net D12: track 68.4 -> 0.00 mm
- net D13: track 64.8 -> 0.00 mm
- net RESET_ARDUINO: track 0.00 -> 56.2 mm
- net RESOLUTION$2: track 356.5 -> 403.2 mm, vias 6 -> 12
- net RESOLUTION$1: track 341.7 -> 388.3 mm, vias 6 -> 12
- net A3: track 117.3 -> 98.4 mm
- net GNDMOT: track 53.3 -> 63.6 mm, vias 0 -> 8
- net A4: track 109.7 -> 100.9 mm
- net DIR$0: track 45.7 -> 51.5 mm
- net DIR$5: track 94.8 -> 89.3 mm
- net STEP$3: track 55.7 -> 50.2 mm
- net STEP$5: track 93.8 -> 88.8 mm
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- added copper zone on layer 1, net NONE
