File: ArduinoUNO_Connexions.sch (EAGLE design)
At the start: 25 parts

Commit message: update
Parts:
- added C10, C9: 0.1 uF, rcl:C-EU025-024X044
- added R13, R14, R15: 1k, rcl:R-US_0207/7
- added R16: 100k, rcl:R-US_0207/7
- added U$5, U$6: BOARD_A4988, Clean-Kong:BOARD_A4988
- C5, C6: value 0.1 uF -> 100uf; device rcl:C-EU025-024X044 -> Seeed-Capacitor:DIP-ALUMINUM-100UF-16V(D5-H7MM)
- R12: value 100k -> 1k
Connections:
- net BSTEP$0 renamed STEP$0
- net BSTEP$1 renamed STEP$1
- net BSTEP$2 renamed STEP$2
- net BSTEP$3 renamed STEP$3
- removed net BDIR$0: PCB2.4, R5.1, U$1.DIR
- removed net BDIR$1: PCB2.~5, R6.1, U$2.DIR
- removed net BDIR$2: PCB2.~6, R7.1, U$3.DIR
- removed net BDIR$3: PCB2.7, R8.1, U$4.DIR
- removed net BRESOLUTION$0: PCB2.~11, R9.1, U$1.MS1, U$2.MS1, U$3.MS1, U$4.MS1
- removed net BRESOLUTION$1: PCB2.12, R10.1, U$1.MS2, U$2.MS2, U$3.MS2, U$4.MS2
- removed net BRESOLUTION$2: PCB2.13, R11.1, U$1.MS3, U$2.MS3, U$3.MS3, U$4.MS3
- new net DIR$0: PCB2.8, R7.2, U$1.DIR
- new net DIR$1: PCB2.~9, R8.2, U$2.DIR
- new net DIR$2: PCB2.~10, R9.2, U$3.DIR
- new net DIR$3: PCB2.~11, R10.2, U$4.DIR
- new net DIR$4: PCB2.12, R11.2, U$5.DIR
- new net DIR$5: PCB2.13, R12.2, U$6.DIR
- new net N$5: R16.2
- new net N$6: U$5.!RESET, U$5.!SLEEP
- new net N$7: U$6.!RESET, U$6.!SLEEP
- new net RESOLUTION$0: PCB2.A0, R15.2
- new net RESOLUTION$1: PCB2.A1, R14.2
- new net RESOLUTION$2: PCB2.A2, R13.2
- new net STEP$17: PCB2.A4, PCB2.A5
- new net STEP$4: PCB2.4, R5.2, U$5.STEP
- new net STEP$5: PCB2.~5, R6.2, U$6.STEP
- net GND: now also C10.1, C5.-, C6.-, C9.1, R10.1, R11.1, R13.1, R14.1, R15.1, R16.1, R5.1, R6.1, R7.1, R8.1, R9.1, U$5.GND, U$5.GNDMOT, U$6.GND, U$6.GNDMOT; no longer C5.1, C6.1, R10.2, R11.2, R12.2, R5.2, R6.2, R7.2, R8.2, R9.2
- net VCC: now also C10.2, C5.+, C6.+, C9.2, U$5.VDD, U$5.VMOT, U$6.VDD, U$6.VMOT; no longer C5.2, C6.2
Other:
- moved on the sheet: C1, C2, C3, C4, C7, C8, R1, R10, R11, R12, R2, R3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

Commit message: update board
Parts:
- added C11, C12: (no value), rcl:C-EU050-030X075
- added D1: (no value), diode:DIODE_SCHOTTKY2-F126-12
- added D2: 1N4004, diode:1N4004
- added JP1, JP10, JP13, JP14, JP17, JP18, JP2, JP21, JP22, JP5, JP6, JP9: (no value), pinhead:PINHD-1X8
- added JP11, JP15, JP19, JP23, JP4, JP7: (no value), pinhead:PINHD-1X2
- added JP12, JP16, JP20, JP24, JP3, JP8: (no value), pinhead:PINHD-1X4
- added LED1, LED2, LED3: (no value), led:LED5MM
- added R17, R18: 250, rcl:R-US_0207/7
- added R19: 2,7K, rcl:R-US_0207/7
- added SV1, SV2: (no value), con-lstb:MA08-1
- added SV3: (no value), con-lstb:MA06-1
- added SV4: (no value), con-lstb:MA10-1
- added X3, X4: (no value), con-ptr500:AK500/2
- C1, C2, C3, C4, C5, C6: value 100uf -> (none); device Seeed-Capacitor:DIP-ALUMINUM-100UF-16V(D5-H7MM) -> rcl:CPOL-EUE5-10.5
- C10, C7, C8, C9: value 0.1 uF -> (none); device rcl:C-EU025-024X044 -> rcl:C-EU050-030X075
Connections:
- removed net STEP$17: PCB2.A4, PCB2.A5
- new net GNDMOT: C1.-, C2.-, C3.-, C4.-, C5.-, C6.-, JP10.2, JP14.2, JP18.2, JP2.2, JP22.2, JP6.2, R16.2, X4-1.KL
- new net N$10: JP1.5, JP4.2
- new net N$11: JP1.6, JP4.1
- new net N$12: JP2.6, JP3.1
- new net N$13: JP5.5, JP7.2
- new net N$14: JP5.6, JP7.1
- new net N$15: JP6.3, JP8.4
- new net N$16: JP6.4, JP8.3
- new net N$17: JP6.5, JP8.2
- new net N$18: JP6.6, JP8.1
- new net N$19: JP11.2, JP9.5
- new net N$20: JP11.1, JP9.6
- new net N$21: JP10.3, JP12.4
- new net N$22: JP10.4, JP12.3
- new net N$23: JP10.5, JP12.2
- new net N$24: JP10.6, JP12.1
- new net N$25: JP13.5, JP15.2
- new net N$26: JP13.6, JP15.1
- new net N$27: JP14.3, JP16.4
- new net N$28: JP14.4, JP16.3
- new net N$29: JP14.5, JP16.2
- new net N$30: JP14.6, JP16.1
- new net N$31: JP17.5, JP19.2
- new net N$32: JP17.6, JP19.1
- new net N$33: JP18.3, JP20.4
- new net N$34: JP18.4, JP20.3
- new net N$35: JP18.5, JP20.2
- new net N$36: JP18.6, JP20.1
- new net N$37: JP21.5, JP23.2
- new net N$38: JP21.6, JP23.1
- new net N$39: JP22.3, JP24.4
- new net N$40: JP22.4, JP24.3
- new net N$41: JP22.5, JP24.2
- new net N$42: JP22.6, JP24.1
- new net N$8: JP2.4, JP3.3
- new net N$9: JP2.5, JP3.2
- new net VMOT: C1.+, C2.+, C3.+, C4.+, C5.+, C6.+, D2.C, JP10.1, JP14.1, JP18.1, JP2.1, JP22.1, JP6.1
- net DIR$0: now also JP1.7, R2.2, SV1.2; no longer PCB2.8, R7.2, U$1.DIR
- net DIR$1: now also JP5.7, R4.2, SV1.4; no longer PCB2.~9, R8.2, U$2.DIR
- net DIR$2: now also JP9.7, R6.2, SV1.6; no longer PCB2.~10, R9.2, U$3.DIR
- net DIR$3: now also JP13.7, R8.2, SV1.8; no longer PCB2.~11, R10.2, U$4.DIR
- net DIR$4: now also JP17.7, R10.2, SV4.2; no longer PCB2.12, R11.2, U$5.DIR
- net DIR$5: now also JP21.7, SV4.4; no longer PCB2.13, U$6.DIR
- net GND: now also C10.2, C11.2, C12.2, C7.2, C8.2, C9.2, JP10.8, JP14.8, JP18.8, JP2.8, JP22.8, JP6.8, R17.1, R18.2, R19.2, SV2.2, SV2.3, SV4.7, X3-1.KL; no longer C1.-, C10.1, C2.-, C3.-, C4.-, C5.-, C6.-, C7.1, C8.1, C9.1, PCB2.GND, PCB2.GND., PCB2.GND.., U$1.GND, U$1.GNDMOT, U$2.GND, U$2.GNDMOT, U$3.GND, U$3.GNDMOT, U$4.GND, U$4.GNDMOT, U$5.GND, U$5.GNDMOT, U$6.GND, U$6.GNDMOT
- net N$1: now also D2.A, LED3.A, X4-2.KL; no longer U$2.!RESET, U$2.!SLEEP
- net N$2: now also D1.2, LED2.A, X3-2.KL; no longer U$1.!RESET, U$1.!SLEEP
- net N$3: now also LED1.A, SV2.5; no longer U$3.!RESET, U$3.!SLEEP
- net N$4: now also LED1.C, R17.2; no longer U$4.!RESET, U$4.!SLEEP
- net N$5: now also JP2.3, JP3.4; no longer R16.2
- net N$6: now also LED3.C, R19.1; no longer U$5.!RESET, U$5.!SLEEP
- net N$7: now also LED2.C, R18.1; no longer U$6.!RESET, U$6.!SLEEP
- net RESOLUTION$0: now also JP1.2, JP13.2, JP17.2, JP21.2, JP5.2, JP9.2, R13.2, SV3.1; no longer PCB2.A0, R15.2
- net RESOLUTION$1: now also JP1.3, JP13.3, JP17.3, JP21.3, JP5.3, JP9.3, SV3.2; no longer PCB2.A1
- net RESOLUTION$2: now also JP1.4, JP13.4, JP17.4, JP21.4, JP5.4, JP9.4, R15.2, SV3.3; no longer PCB2.A2, R13.2
- net STEP$0: now also JP1.8, SV1.1; no longer PCB2.0(RX), U$1.STEP
- net STEP$1: now also JP5.8, R3.2, SV1.3; no longer PCB2.1(TX), R2.2, U$2.STEP
- net STEP$2: now also JP9.8, R5.2, SV1.5; no longer PCB2.2, R3.2, U$3.STEP
- net STEP$3: now also JP13.8, R7.2, SV1.7; no longer PCB2.~3, R4.2, U$4.STEP
- net STEP$4: now also JP17.8, R9.2, SV4.1; no longer PCB2.4, R5.2, U$5.STEP
- net STEP$5: now also JP21.8, R11.2, SV4.3; no longer PCB2.~5, R6.2, U$6.STEP
- net VCC: now also C10.1, C11.1, C12.1, C7.1, C8.1, C9.1, D1.1, JP10.7, JP14.7, JP18.7, JP2.7, JP22.7, JP6.7; no longer C1.+, C10.2, C2.+, C3.+, C4.+, C5.+, C6.+, C7.2, C8.2, C9.2, PCB2.5V, U$1.VDD, U$1.VMOT, U$2.VDD, U$2.VMOT, U$3.VDD, U$3.VMOT, U$4.VDD, U$4.VMOT, U$5.VDD, U$5.VMOT, U$6.VDD, U$6.VMOT
Other:
- note added: "Connect the Raspberry pi via USB"
- note added: "Put as close as possible of the VMOT and GNDMOT supply pin of the drivers"
- note added: "VCC = 5V"
- note removed: "USB TO RASPBERRY PI ->"
- moved on the sheet: C10, C7, C8, C9, R1, R10, R11, R12, R13, R14, R15, R16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

Commit message: update with new guidlines
Parts:
- added D3, D4, D5: 1N4004, diode:1N4004
- added R20, R21, R22, R23, R24: 1k, rcl:R-US_0207/7
- added SV5: (no value), con-lstb:MA05-1
- added X1: (no value), con-ptr500:AK500/2
- R16: value 100k -> 0
Connections:
- new net A3: R22.1, SV3.4, SV5.3
- new net A4: R23.1, SV3.5, SV5.4
- new net A5: R24.1, SV3.6, SV5.5
- new net D12: R20.2, SV4.5, SV5.1
- new net D13: R21.2, SV4.6, SV5.2
- new net N$56: D4.A, D5.A, X1-2.KL
- net DIR$0: now also R1.2, SV1.1; no longer R2.2, SV1.2
- net DIR$1: now also R3.2, SV1.3; no longer R4.2, SV1.4
- net DIR$2: now also R5.2, SV1.5; no longer R6.2, SV1.6
- net DIR$3: now also R7.2, SV1.7; no longer R8.2, SV1.8
- net DIR$4: now also R9.2, SV4.1; no longer R10.2, SV4.2
- net DIR$5: now also R11.2, SV4.3; no longer R12.2, SV4.4
- net GND: now also R20.1, R21.1, R22.2, R23.2, R24.2
- net GNDMOT: now also X1-1.KL
- net N$1: now also D3.A; no longer LED3.A
- net N$2: now also D1.1; no longer D1.2
- net STEP$0: now also R2.2, SV1.2; no longer R1.2, SV1.1
- net STEP$1: now also R4.2, SV1.4; no longer R3.2, SV1.3
- net STEP$2: now also R6.2, SV1.6; no longer R5.2, SV1.5
- net STEP$3: now also R8.2, SV1.8; no longer R7.2, SV1.7
- net STEP$4: now also R10.2, SV4.2; no longer R9.2, SV4.1
- net STEP$5: now also R12.2, SV4.4; no longer R11.2, SV4.3
- net VCC: now also D1.2; no longer D1.1
- net VMOT: now also D3.C, D4.C, D5.C, LED3.A
Other:
- note added: "Possibility to put 2 diodes"
- note added: "Unused ports"
- moved on the sheet: D1, LED3, R1, R10, R11, R12, R16, R19, R2, R3, R4, R5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

Commit message: Final update before printing first prototype
Parts:
- added S1: (no value), switch:255SB
Connections:
- new net N$43: S1.P, SV2.1
- net VCC: now also S1.O
Changed lines of the file:
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@@
 <part name="SUPPLY19" library="supply2" library_urn="urn:adsk.eagle:library:372" deviceset="GND" device=""/>
 <part name="D1" library="diode" library_urn="urn:adsk.eagle:library:210" deviceset="DIODE_SCHOTTKY2-" device="F126-12" package3d_urn="urn:adsk.eagle:package:43358/1"/>
+<part name="P+2" library="supply1" library_urn="urn:adsk.eagle:library:371" deviceset="VCC" device=""/>
+<part name="S1" library="switch" library_urn="urn:adsk.eagle:library:380" deviceset="255SB" device="" package3d_urn="urn:adsk.eagle:package:27679/1">
+<variant name="Actual" populate="no"/>
+</part>
 </parts>
 <sheets>
@@
 <attribute name="NAME" x="603.25" y="158.115" size="1.778" layer="95" rot="R180"/>
 <attribute name="VALUE" x="598.17" y="158.369" size="1.778" layer="96" rot="R180"/>
+</instance>
+<instance part="P+2" gate="VCC" x="543.56" y="213.36" smashed="yes">
+<attribute name="VALUE" x="546.1" y="213.36" size="1.778" layer="96"/>
+</instance>
+<instance part="S1" gate="1" x="535.94" y="208.28" smashed="yes" rot="R270">
+<attribute name="NAME" x="528.955" y="209.55" size="1.778" layer="95"/>
+<attribute name="VALUE" x="539.115" y="212.09" size="1.778" layer="96"/>
 </instance>
 </instances>
@@
 <pinref part="D1" gate="G$1" pin="2"/>
 </segment>
+<segment>
+<pinref part="P+2" gate="VCC" pin="VCC"/>
+<wire x1="543.56" y1="210.82" x2="543.56" y2="208.28" width="0.1524" layer="91"/>
+<pinref part="S1" gate="1" pin="O"/>
+<wire x1="541.02" y1="208.28" x2="543.56" y2="208.28" width="0.1524" layer="91"/>
+</segment>
 </net>
 <net name="STEP$0" class="0">
@@
 </segment>
 </net>
+<net name="N$43" class="0">
+<segment>
+<pinref part="SV2" gate="1" pin="1"/>
+<wire x1="485.14" y1="205.74" x2="530.86" y2="205.74" width="0.1524" layer="91"/>
+<pinref part="S1" gate="1" pin="P"/>
+</segment>
+</net>

Commit message: Update
Parts:
- added D6: (no value), diode:DIODE_SCHOTTKY2-F126-12
- added X2: (no value), con-ptr500:AK500/2
Connections:
- new net ALIM_ARDUINO: D6.2, S1.O
- new net N$44: D6.1, X2-2.KL
- net GND: now also X2-1.KL
- net VCC: no longer S1.O
Other:
- moved on the sheet: D1, D2, D3, D4, D5, LED2, LED3, R16, R18, R19, X1-1, X1-2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

Commit message: update
Parts:
- removed PCB2: ARDUINO_UNO, E14_Arduino_revC:ARDUINO_UNO
- removed U$1, U$2, U$3, U$4, U$5, U$6: BOARD_A4988, Clean-Kong:BOARD_A4988
Changed lines of the file:
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@@
 </classes>
 <parts>
-<part name="PCB2" library="E14_Arduino_revC" deviceset="ARDUINO_UNO" device="">
-<variant name="Actual" populate="no"/>
-</part>
 <part name="R1" library="rcl" library_urn="urn:adsk.eagle:library:334" deviceset="R-US_" device="0207/7" package3d_urn="urn:adsk.eagle:package:23493/1" value="1k"/>
 <part name="SUPPLY15" library="supply2" library_urn="urn:adsk.eagle:library:372" deviceset="GND" device=""/>
@@
 <attribute name="AMPS" value="15"/>
 </part>
-<part name="U$1" library="Clean-Kong" deviceset="BOARD_A4988" device="">
-<variant name="Actual" populate="no"/>
-</part>
-<part name="U$2" library="Clean-Kong" deviceset="BOARD_A4988" device="">
-<variant name="Actual" populate="no"/>
-</part>
-<part name="U$3" library="Clean-Kong" deviceset="BOARD_A4988" device="">
-<variant name="Actual" populate="no"/>
-</part>
-<part name="U$4" library="Clean-Kong" deviceset="BOARD_A4988" device="">
-<variant name="Actual" populate="no"/>
-</part>
-<part name="U$5" library="Clean-Kong" deviceset="BOARD_A4988" device="">
-<variant name="Actual" populate="no"/>
-</part>
-<part name="U$6" library="Clean-Kong" deviceset="BOARD_A4988" device="">
-<variant name="Actual" populate="no"/>
-</part>
 <part name="LED1" library="led" library_urn="urn:adsk.eagle:library:259" deviceset="LED" device="5MM" package3d_urn="urn:adsk.eagle:package:15799/2"/>
 <part name="LED2" library="led" library_urn="urn:adsk.eagle:library:259" deviceset="LED" device="5MM" package3d_urn="urn:adsk.eagle:package:15799/2"/>
@@
 </plain>
 <instances>
-<instance part="PCB2" gate="G$1" x="576.58" y="271.78" smashed="yes" rot="R180"/>
 <instance part="R1" gate="G$1" x="530.86" y="363.22" smashed="yes" rot="R180">
 <attribute name="NAME" x="534.67" y="361.7214" size="1.778" layer="95" rot="R180"/>
@@
 <attribute name="VALUE" x="520.7" y="136.9314" size="1.778" layer="96" rot="R180" display="off"/>
 </instance>
-<instance part="U$1" gate="G$1" x="403.86" y="53.34" smashed="yes">
-<attribute name="NAME" x="424.18" y="73.66" size="2.54" layer="95"/>
-</instance>
-<instance part="U$2" gate="G$1" x="525.78" y="53.34" smashed="yes">
-<attribute name="NAME" x="546.1" y="73.66" size="2.54" layer="95"/>
-</instance>
-<instance part="U$3" gate="G$1" x="403.86" y="-27.94" smashed="yes">
-<attribute name="NAME" x="424.18" y="-7.62" size="2.54" layer="95"/>
-</instance>
-<instance part="U$4" gate="G$1" x="528.32" y="-27.94" smashed="yes">
-<attribute name="NAME" x="548.64" y="-7.62" size="2.54" layer="95"/>
-</instance>
-<instance part="U$5" gate="G$1" x="406.4" y="-111.76" smashed="yes">
-<attribute name="NAME" x="426.72" y="-91.44" size="2.54" layer="95"/>
-</instance>
-<instance part="U$6" gate="G$1" x="530.86" y="-111.76" smashed="yes">
-<attribute name="NAME" x="551.18" y="-91.44" size="2.54" layer="95"/>
-</instance>
 <instance part="LED1" gate="G$1" x="490.22" y="195.58" smashed="yes" rot="R90">

Commit message: update
Other:
- note added: "Connectors for the Arduino UNO"
- note added: "Connectors for the drivers"
- moved on the sheet: C1, C10, C11, C12, C2, C3, C4, C5, C6, C7, C8, C9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

Commit message: update
Parts:
- removed R20, R21: 1k, rcl:R-US_0207/7
- added S2: (no value), switch-omron:10-XX
- C1, C2, C3, C4, C5, C6: value (none) -> 100uF
- C10, C11, C12, C7, C8, C9: value (none) -> 0,1uF
- D2, D3, D4, D5: value 1N4004 -> 1N5400; device diode:1N4004 -> diode:1N5400; AMPS 15 -> (none)
- R17, R18: value 250 -> 125
- R19: value 2,7K -> 1,4K
- SV5: device con-lstb:MA05-1 -> con-lstb:MA03-1
Connections:
- net N$43 renamed VIN_ARDUINO
- removed net D12: R20.2, SV4.5, SV5.1
- removed net D13: R21.2, SV4.6, SV5.2
- removed net N$3: LED1.A, SV2.5
- new net 3V3_ARDUINO: SV2.5
- new net 5V_ARDUINO: LED1.A, SV2.4
- new net IOREF_ARDUINO: SV2.7
- new net RESET_ARDUINO: S2.P, S2.P1, SV2.6
- new net RX_ARDUINO: SV1.1
- new net TX_ARDUINO: SV1.2
- net A4: now also SV5.2; no longer SV5.4
- net A5: now also SV5.1; no longer SV5.5
- net DIR$0: now also SV1.3; no longer SV1.1
- net DIR$1: now also SV1.5; no longer SV1.3
- net DIR$2: now also SV1.7; no longer SV1.5
- net DIR$3: now also SV4.1; no longer SV1.7
- net DIR$4: now also SV4.3; no longer SV4.1
- net DIR$5: now also SV4.5; no longer SV4.3
- net GND: now also S2.S, S2.S1; no longer R20.1, R21.1
- net N$1: now also D4.A, D5.A; no longer D2.A, D3.A
- net N$56: now also D2.A, D3.A; no longer D4.A, D5.A
- net STEP$0: now also SV1.4; no longer SV1.2
- net STEP$1: now also SV1.6; no longer SV1.4
- net STEP$2: now also SV1.8; no longer SV1.6
- net STEP$3: now also SV4.2; no longer SV1.8
- net STEP$4: now also SV4.4; no longer SV4.2
- net STEP$5: now also SV4.6; no longer SV4.4
Other:
- note added: "Connectors for the a4988 drivers"
- note added: "Imax = 2A (for one a4988 driver) * 6 = 12A But, this is the current going through the stepper motor after the voltage conversion. The current needed by the source is less than this: Pstepper = 2,5V*2A = 5W Isrc = 5W/24V => Isrc = 4,8A"
- note added: "Only connected the 2 gnd in one point"
- note added: "Pull down resistors"
- note added: "Shortkey diode"
- note removed: "Connectors for the drivers"
- note removed: "Only connected in one point"
- moved on the sheet: C1, C10, C11, C12, C2, C3, C4, C5, C6, C7, C8, C9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
