File: RaspberryPi_Connections.sch (EAGLE design)
At the start: 3 parts

Commit message: update
Parts:
- removed J1: (no value), con-amp:MTA05-100
- added JP1: (no value), pinhead:PINHD-1X7
- added JP2: (no value), pinhead:PINHD-1X5
- U$1: value MCP3201-CI/SN -> MCP3201-CI/P; device MCP3201-CI_SN:MCP3201-CI/SN -> MCP3201-CI_P:MCP3201-CI/P
Connections:
- new net CEO_A: JP1.4
- net 5V_RPI: now also JP1.1, JP2.1; no longer J1.1, PCB1.5V@2
- net CE0_A: no longer PCB1.GPIO8
- net GND_RPI: now also JP1.7, JP2.5; no longer J1.5, PCB1.GND@6
- net MISO_A: now also JP1.5; no longer PCB1.GPIO9
- net SCLK_A: now also JP1.6; no longer PCB1.GPIO11
- net TOOL_CHANGER_ANALOG_I: now also JP2.4; no longer J1.4
- net TOOL_CHANGER_DIGITAL_I: now also JP1.2, JP2.2; no longer J1.2, PCB1.GPIO23
- net TOOL_CHANGER_DIGITAL_O: now also JP1.3, JP2.3; no longer J1.3, PCB1.GPIO24
Other:
- note added: "Signals enter in board from raspberry pi by the pin headers"
- note added: "TOOL_CHANGER_DIGITAL_I to BCM 23 on Raspberry Pi TOOL_CHANGER_DIGITAL_O to BCM 24 on Raspberry Pi CEO_A to BCM 08 on Raspberry Pi MISO_A to BCM 09 on Raspberry Pi SCLK_A to BCM 11 on Raspberry Pi"
- moved on the sheet: U$1

Commit message: update
Parts:
- removed PCB1: RPI2, e14_Rpi2_RevA:RPI2
Changed lines of the file:
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@@
 </classes>
 <parts>
-<part name="PCB1" library="e14_Rpi2_RevA" deviceset="RPI2" device=""/>
 <part name="JP2" library="pinhead" library_urn="urn:adsk.eagle:library:325" deviceset="PINHD-1X5" device="" package3d_urn="urn:adsk.eagle:package:22469/2"/>
 <part name="JP1" library="pinhead" library_urn="urn:adsk.eagle:library:325" deviceset="PINHD-1X7" device="" package3d_urn="urn:adsk.eagle:package:22477/2"/>
@@
 </plain>
 <instances>
-<instance part="PCB1" gate="G$1" x="10.16" y="78.74" smashed="yes"/>
 <instance part="JP2" gate="A" x="236.22" y="220.98" smashed="yes">
 <attribute name="NAME" x="229.87" y="229.235" size="1.778" layer="95"/>

Commit message: update
Other:
- note removed: "USB0 TO ARDUINO -> USB1 TO WEBCAM -> USB2 TO WIRELESS MODULE -> USB3 TO (UNUSED) ->"
- moved on the sheet: JP2
Changed lines of the file:
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@@
 <sheet>
 <plain>
-<text x="177.8" y="144.78" size="1.778" layer="91">USB0 TO ARDUINO -&gt;
-USB1 TO WEBCAM -&gt;
-USB2 TO WIRELESS MODULE -&gt;
-USB3 TO (UNUSED) -&gt;</text>
-<text x="198.12" y="231.14" size="1.778" layer="91">TOOL CHANGER CONNECTOR-&gt;</text>
+<text x="114.3" y="180.34" size="1.778" layer="91">TOOL CHANGER CONNECTOR-&gt;</text>
 <text x="139.7" y="241.3" size="1.778" layer="91">ANALOG INPUT</text>
 <text x="27.94" y="241.3" size="1.778" layer="91">Signals enter in board from raspberry pi by the pin headers</text>
@@
 </plain>
 <instances>
-<instance part="JP2" gate="A" x="236.22" y="220.98" smashed="yes">
-<attribute name="NAME" x="229.87" y="229.235" size="1.778" layer="95"/>
-<attribute name="VALUE" x="229.87" y="210.82" size="1.778" layer="96"/>
+<instance part="JP2" gate="A" x="152.4" y="170.18" smashed="yes">
+<attribute name="NAME" x="146.05" y="178.435" size="1.778" layer="95"/>
+<attribute name="VALUE" x="146.05" y="160.02" size="1.778" layer="96"/>
 </instance>
 <instance part="JP1" gate="A" x="17.78" y="223.52" smashed="yes" rot="MR0">
@@
 </segment>
 <segment>
-<wire x1="233.68" y1="226.06" x2="193.04" y2="226.06" width="0.1524" layer="91"/>
-<label x="193.04" y="226.06" size="1.778" layer="95"/>
+<wire x1="149.86" y1="175.26" x2="109.22" y2="175.26" width="0.1524" layer="91"/>
+<label x="109.22" y="175.26" size="1.778" layer="95"/>
 <pinref part="JP2" gate="A" pin="1"/>
 </segment>
@@
 </segment>
 <segment>
-<wire x1="233.68" y1="215.9" x2="193.04" y2="215.9" width="0.1524" layer="91"/>
-<label x="193.04" y="215.9" size="1.778" layer="95"/>
+<wire x1="149.86" y1="165.1" x2="109.22" y2="165.1" width="0.1524" layer="91"/>
+<label x="109.22" y="165.1" size="1.778" layer="95"/>
 <pinref part="JP2" gate="A" pin="5"/>
 </segment>
@@
 </segment>
 <segment>
-<wire x1="233.68" y1="218.44" x2="193.04" y2="218.44" width="0.1524" layer="91"/>
-<label x="193.04" y="218.44" size="1.778" layer="95"/>
+<wire x1="149.86" y1="167.64" x2="109.22" y2="167.64" width="0.1524" layer="91"/>
+<label x="109.22" y="167.64" size="1.778" layer="95"/>
 <pinref part="JP2" gate="A" pin="4"/>
 </segment>
@@
 <net name="TOOL_CHANGER_DIGITAL_O" class="0">
 <segment>
-<wire x1="233.68" y1="220.98" x2="193.04" y2="220.98" width="0.1524" layer="91"/>
-<label x="193.04" y="220.98" size="1.778" layer="95"/>
+<wire x1="149.86" y1="170.18" x2="109.22" y2="170.18" width="0.1524" layer="91"/>
+<label x="109.22" y="170.18" size="1.778" layer="95"/>
 <pinref part="JP2" gate="A" pin="3"/>
 </segment>
@@
 <net name="TOOL_CHANGER_DIGITAL_I" class="0">
 <segment>
-<wire x1="233.68" y1="223.52" x2="193.04" y2="223.52" width="0.1524" layer="91"/>
-<label x="193.04" y="223.52" size="1.778" layer="95"/>
+<wire x1="149.86" y1="172.72" x2="109.22" y2="172.72" width="0.1524" layer="91"/>
+<label x="109.22" y="172.72" size="1.778" layer="95"/>
 <pinref part="JP2" gate="A" pin="2"/>
 </segment>
